Commit message: edit juliet

File: crowdbotsim/JulietteY20MP_crowdbotsim1.urdf (robot description, URDF)
Before this commit: robot JulietteY20MP_crowdbotsim, 56 links, 55 joints
Links:
- added link BumperB_frame, mass 1E-07
- added link BumperFL_frame, mass 1E-07
- added link BumperFR_frame, mass 1E-07
- added link CameraBottom_frame, mass 1E-07
- added link CameraBottom_optical_frame, mass 1E-07
- added link CameraDepth_frame, mass 1E-07
- added link CameraDepth_optical_frame, mass 1E-07
- added link CameraTop_frame, mass 1E-07
- added link CameraTop_optical_frame, mass 1E-07
- added link ChestButton_frame, mass 1E-07
- added link HeadPitch_ears, mass 1E-07; visual mesh filename=package://crowdbotsim/meshes/HeadPitch_ears.stl scale=0.1 0.1 0.1
- added link HeadPitch_milky, mass 1E-07; visual mesh filename=package://crowdbotsim/meshes/HeadPitch_milky.stl scale=0.1 0.1 0.1
- added link HeadPitch_shiny, mass 1E-07; visual mesh filename=package://crowdbotsim/meshes/HeadPitch_shiny.stl scale=0.1 0.1 0.1
- added link HeadTouchFront_frame, mass 1E-07
- added link HeadTouchMiddle_frame, mass 1E-07
- added link HeadTouchRear_frame, mass 1E-07
- added link HipPitch_shiny, mass 1E-07; visual mesh filename=package://crowdbotsim/meshes/HipPitch_shiny.stl scale=0.1 0.1 0.1
- added link ImuBaseAccelerometer_frame, mass 1E-07
- added link ImuTorsoAccelerometer_frame, mass 1E-07
- added link ImuTorsoGyrometer_frame, mass 1E-07
- added link KneePitch_milky, mass 1E-07; visual mesh filename=package://crowdbotsim/meshes/KneePitch_milky.stl scale=0.1 0.1 0.1
- added link LElbowRoll_milky, mass 1E-07; visual mesh filename=package://crowdbotsim/meshes/LElbowRoll_milky.stl scale=0.1 0.1 0.1
- added link LHandTouchBack_frame, mass 1E-07
- added link LShoulderRoll_shiny, mass 1E-07; visual mesh filename=package://crowdbotsim/meshes/LShoulderRoll_shiny.stl scale=0.1 0.1 0.1
- added link LSpeaker_frame, mass 1E-07
- added link RSpeaker_frame, mass 1E-07
- added link ShovelLaser_frame, mass 1E-07
- added link SonarBack_frame, mass 1E-07
- added link SonarFront_frame, mass 1E-07
- added link SurroundingFrontLaser_device_frame, mass 1E-07
- added link SurroundingFrontLaser_frame, mass 1E-07
- added link SurroundingLeftLaser_device_frame, mass 1E-07
- added link SurroundingLeftLaser_frame, mass 1E-07
- added link SurroundingRightLaser_device_frame, mass 1E-07
- added link SurroundingRightLaser_frame, mass 1E-07
- added link Tablet_frame, mass 1E-07
- added link Torso_shiny, mass 1E-07; visual mesh filename=package://crowdbotsim/meshes/Torso_shiny.stl scale=0.1 0.1 0.1
- added link Torso_transparent, mass 1E-07; visual mesh filename=package://crowdbotsim/meshes/Torso_transparent.stl scale=0.1 0.1 0.1
- added link VerticalLeftLaser_frame, mass 1E-07
- added link VerticalRightLaser_frame, mass 1E-07
- link Head: geometry collision mesh filename=package://crowdbotsim/meshes/HeadPitch_0.10.stl scale=0.1 0.1 0.1; visual mesh filename=package://crowdbotsim/meshes/HeadPitch_eyes.stl scale=0.1 0.1 0.1
- link Hip: geometry collision mesh filename=package://crowdbotsim/meshes/HipRoll_0.10.stl scale=0.1 0.1 0.1; visual mesh filename=package://crowdbotsim/meshes/HipRoll.stl scale=0.1 0.1 0.1
- link LBicep: geometry collision mesh filename=package://crowdbotsim/meshes/LShoulderRoll_0.10.stl scale=0.1 0.1 0.1; visual mesh filename=package://crowdbotsim/meshes/LShoulderRoll_milky.stl scale=0.1 0.1 0.1
- link LElbow: geometry collision mesh filename=package://crowdbotsim/meshes/LElbowYaw_0.10.stl scale=0.1 0.1 0.1; visual mesh filename=package://crowdbotsim/meshes/LElbowYaw.stl scale=0.1 0.1 0.1
- link LFinger11_link: geometry collision mesh filename=package://crowdbotsim/meshes/LFinger11.stl scale=0.1 0.1 0.1; visual mesh filename=package://crowdbotsim/meshes/LFinger11.stl scale=0.1 0.1 0.1
- link LFinger12_link: geometry collision mesh filename=package://crowdbotsim/meshes/LFinger12.stl scale=0.1 0.1 0.1; visual mesh filename=package://crowdbotsim/meshes/LFinger12.stl scale=0.1 0.1 0.1
- link LFinger13_link: geometry collision mesh filename=package://crowdbotsim/meshes/LFinger13.stl scale=0.1 0.1 0.1; visual mesh filename=package://crowdbotsim/meshes/LFinger13.stl scale=0.1 0.1 0.1
- link LFinger21_link: geometry collision mesh filename=package://crowdbotsim/meshes/LFinger21.stl scale=0.1 0.1 0.1; visual mesh filename=package://crowdbotsim/meshes/LFinger21.stl scale=0.1 0.1 0.1
- link LFinger22_link: geometry collision mesh filename=package://crowdbotsim/meshes/LFinger22.stl scale=0.1 0.1 0.1; visual mesh filename=package://crowdbotsim/meshes/LFinger22.stl scale=0.1 0.1 0.1
- link LFinger23_link: geometry collision mesh filename=package://crowdbotsim/meshes/LFinger23.stl scale=0.1 0.1 0.1; visual mesh filename=package://crowdbotsim/meshes/LFinger23.stl scale=0.1 0.1 0.1
- link LFinger31_link: geometry collision mesh filename=package://crowdbotsim/meshes/LFinger31.stl scale=0.1 0.1 0.1; visual mesh filename=package://crowdbotsim/meshes/LFinger31.stl scale=0.1 0.1 0.1
- link LFinger32_link: geometry collision mesh filename=package://crowdbotsim/meshes/LFinger32.stl scale=0.1 0.1 0.1; visual mesh filename=package://crowdbotsim/meshes/LFinger32.stl scale=0.1 0.1 0.1
- link LFinger33_link: geometry collision mesh filename=package://crowdbotsim/meshes/LFinger33.stl scale=0.1 0.1 0.1; visual mesh filename=package://crowdbotsim/meshes/LFinger33.stl scale=0.1 0.1 0.1
- link LFinger41_link: geometry collision mesh filename=package://crowdbotsim/meshes/LFinger41.stl scale=0.1 0.1 0.1; visual mesh filename=package://crowdbotsim/meshes/LFinger41.stl scale=0.1 0.1 0.1
- link LFinger42_link: geometry collision mesh filename=package://crowdbotsim/meshes/LFinger42.stl scale=0.1 0.1 0.1; visual mesh filename=package://crowdbotsim/meshes/LFinger42.stl scale=0.1 0.1 0.1
- link LFinger43_link: geometry collision mesh filename=package://crowdbotsim/meshes/LFinger43.stl scale=0.1 0.1 0.1; visual mesh filename=package://crowdbotsim/meshes/LFinger43.stl scale=0.1 0.1 0.1
- link LForeArm: geometry collision mesh filename=package://crowdbotsim/meshes/LElbowRoll_0.10.stl scale=0.1 0.1 0.1; visual mesh filename=package://crowdbotsim/meshes/LElbowRoll_shiny.stl scale=0.1 0.1 0.1
- link LShoulder: geometry collision mesh filename=package://crowdbotsim/meshes/LShoulderPitch_0.10.stl scale=0.1 0.1 0.1; visual mesh filename=package://crowdbotsim/meshes/LShoulderPitch.stl scale=0.1 0.1 0.1
- link LThumb1_link: geometry collision mesh filename=package://crowdbotsim/meshes/LThumb1.stl scale=0.1 0.1 0.1; visual mesh filename=package://crowdbotsim/meshes/LThumb1.stl scale=0.1 0.1 0.1
- link LThumb2_link: geometry collision mesh filename=package://crowdbotsim/meshes/LThumb2.stl scale=0.1 0.1 0.1; visual mesh filename=package://crowdbotsim/meshes/LThumb2.stl scale=0.1 0.1 0.1
- link Neck: geometry collision mesh filename=package://crowdbotsim/meshes/HeadYaw_0.10.stl scale=0.1 0.1 0.1; visual mesh filename=package://crowdbotsim/meshes/HeadYaw.stl scale=0.1 0.1 0.1
- link Pelvis: geometry collision mesh filename=package://crowdbotsim/meshes/HipPitch_0.10.stl scale=0.1 0.1 0.1; visual mesh filename=package://crowdbotsim/meshes/HipPitch_milky.stl scale=0.1 0.1 0.1
- link RBicep: geometry collision mesh filename=package://crowdbotsim/meshes/RShoulderRoll_0.10.stl scale=0.1 0.1 0.1; visual mesh filename=package://crowdbotsim/meshes/RShoulderRoll_milky.stl scale=0.1 0.1 0.1
- link RElbow: geometry collision mesh filename=package://crowdbotsim/meshes/RElbowYaw_0.10.stl scale=0.1 0.1 0.1; visual mesh filename=package://crowdbotsim/meshes/RElbowYaw.stl scale=0.1 0.1 0.1
- link RElbowRoll_milky: mass 1E-05 -> 1E-07; geometry visual mesh filename=package://crowdbotsim/meshes/RElbowRoll_milky.stl scale=0.1 0.1 0.1
- link RFinger11_link: geometry collision mesh filename=package://crowdbotsim/meshes/RFinger11.stl scale=0.1 0.1 0.1; visual mesh filename=package://crowdbotsim/meshes/RFinger11.stl scale=0.1 0.1 0.1
- link RFinger12_link: geometry collision mesh filename=package://crowdbotsim/meshes/RFinger12.stl scale=0.1 0.1 0.1; visual mesh filename=package://crowdbotsim/meshes/RFinger12.stl scale=0.1 0.1 0.1
- link RFinger13_link: geometry collision mesh filename=package://crowdbotsim/meshes/RFinger13.stl scale=0.1 0.1 0.1; visual mesh filename=package://crowdbotsim/meshes/RFinger13.stl scale=0.1 0.1 0.1
- link RFinger21_link: geometry collision mesh filename=package://crowdbotsim/meshes/RFinger21.stl scale=0.1 0.1 0.1; visual mesh filename=package://crowdbotsim/meshes/RFinger21.stl scale=0.1 0.1 0.1
- link RFinger22_link: geometry collision mesh filename=package://crowdbotsim/meshes/RFinger22.stl scale=0.1 0.1 0.1; visual mesh filename=package://crowdbotsim/meshes/RFinger22.stl scale=0.1 0.1 0.1
- link RFinger23_link: geometry collision mesh filename=package://crowdbotsim/meshes/RFinger23.stl scale=0.1 0.1 0.1; visual mesh filename=package://crowdbotsim/meshes/RFinger23.stl scale=0.1 0.1 0.1
- link RFinger31_link: geometry collision mesh filename=package://crowdbotsim/meshes/RFinger31.stl scale=0.1 0.1 0.1; visual mesh filename=package://crowdbotsim/meshes/RFinger31.stl scale=0.1 0.1 0.1
- link RFinger32_link: geometry collision mesh filename=package://crowdbotsim/meshes/RFinger32.stl scale=0.1 0.1 0.1; visual mesh filename=package://crowdbotsim/meshes/RFinger32.stl scale=0.1 0.1 0.1
- link RFinger33_link: geometry collision mesh filename=package://crowdbotsim/meshes/RFinger33.stl scale=0.1 0.1 0.1; visual mesh filename=package://crowdbotsim/meshes/RFinger33.stl scale=0.1 0.1 0.1
- link RFinger41_link: geometry collision mesh filename=package://crowdbotsim/meshes/RFinger41.stl scale=0.1 0.1 0.1; visual mesh filename=package://crowdbotsim/meshes/RFinger41.stl scale=0.1 0.1 0.1
- link RFinger42_link: geometry collision mesh filename=package://crowdbotsim/meshes/RFinger42.stl scale=0.1 0.1 0.1; visual mesh filename=package://crowdbotsim/meshes/RFinger42.stl scale=0.1 0.1 0.1
- link RFinger43_link: geometry collision mesh filename=package://crowdbotsim/meshes/RFinger43.stl scale=0.1 0.1 0.1; visual mesh filename=package://crowdbotsim/meshes/RFinger43.stl scale=0.1 0.1 0.1
- link RForeArm: geometry collision mesh filename=package://crowdbotsim/meshes/RElbowRoll_0.10.stl scale=0.1 0.1 0.1; visual mesh filename=package://crowdbotsim/meshes/RElbowRoll_shiny.stl scale=0.1 0.1 0.1
- link RHandTouchBack_frame: mass 1E-05 -> 1E-07
- link RShoulder: geometry collision mesh filename=package://crowdbotsim/meshes/RShoulderPitch_0.10.stl scale=0.1 0.1 0.1; visual mesh filename=package://crowdbotsim/meshes/RShoulderPitch.stl scale=0.1 0.1 0.1
- link RShoulderRoll_shiny: mass 1E-05 -> 1E-07; geometry visual mesh filename=package://crowdbotsim/meshes/RShoulderRoll_shiny.stl scale=0.1 0.1 0.1
- link RThumb1_link: geometry collision mesh filename=package://crowdbotsim/meshes/RThumb1.stl scale=0.1 0.1 0.1; visual mesh filename=package://crowdbotsim/meshes/RThumb1.stl scale=0.1 0.1 0.1
- link RThumb2_link: geometry collision mesh filename=package://crowdbotsim/meshes/RThumb2.stl scale=0.1 0.1 0.1; visual mesh filename=package://crowdbotsim/meshes/RThumb2.stl scale=0.1 0.1 0.1
- link Tibia: geometry collision mesh filename=package://crowdbotsim/meshes/KneePitch_0.10.stl scale=0.1 0.1 0.1; visual mesh filename=package://crowdbotsim/meshes/KneePitch_shiny.stl scale=0.1 0.1 0.1
- link WheelB_link: geometry collision mesh filename=package://crowdbotsim/meshes/WheelB_0.10.stl scale=0.1 0.1 0.1; visual mesh filename=package://crowdbotsim/meshes/WheelB.stl scale=0.1 0.1 0.1
- link WheelFL_link: geometry collision mesh filename=package://crowdbotsim/meshes/WheelFL_0.10.stl scale=0.1 0.1 0.1; visual mesh filename=package://crowdbotsim/meshes/WheelFL.stl scale=0.1 0.1 0.1
- link WheelFR_link: geometry collision mesh filename=package://crowdbotsim/meshes/WheelFR_0.10.stl scale=0.1 0.1 0.1; visual mesh filename=package://crowdbotsim/meshes/WheelFR.stl scale=0.1 0.1 0.1
- link base_footprint: mass 0.001 -> 1E-07
- link base_link: mass 0.001 -> 1E-07
- link l_wrist: geometry collision mesh filename=package://crowdbotsim/meshes/LWristYaw.stl scale=0.1 0.1 0.1; visual mesh filename=package://crowdbotsim/meshes/LWristYaw.stl scale=0.1 0.1 0.1
- link r_wrist: geometry collision mesh filename=package://crowdbotsim/meshes/RWristYaw.stl scale=0.1 0.1 0.1; visual mesh filename=package://crowdbotsim/meshes/RWristYaw.stl scale=0.1 0.1 0.1
- link sick_laser_front: mass 1E-05 -> 0.1000000015
- link sick_laser_rear: mass 1E-05 -> 0.1000000015
- link torso: geometry collision mesh filename=package://crowdbotsim/meshes/Torso_0.10.stl scale=0.1 0.1 0.1; visual mesh filename=package://crowdbotsim/meshes/Torso_milky.stl scale=0.1 0.1 0.1
Joints:
- removed joint Hip_torso_joint
- removed joint LBicep_LElbow_joint
- removed joint LElbow_LForeArm_joint
- removed joint LFinger11_link_LFinger12_link_joint
- removed joint LFinger12_link_LFinger13_link_joint
- removed joint LFinger21_link_LFinger22_link_joint
- removed joint LFinger22_link_LFinger23_link_joint
- removed joint LFinger31_link_LFinger32_link_joint
- removed joint LFinger32_link_LFinger33_link_joint
- removed joint LFinger41_link_LFinger42_link_joint
- removed joint LFinger42_link_LFinger43_link_joint
- removed joint LForeArm_l_wrist_joint
- removed joint LShoulder_LBicep_joint
- removed joint LThumb1_link_LThumb2_link_joint
- removed joint Neck_Head_joint
- removed joint Pelvis_Hip_joint
- removed joint RBicep_RElbow_joint
- removed joint RBicep_RShoulderRoll_shiny_joint
- removed joint RElbow_RForeArm_joint
- removed joint RFinger11_link_RFinger12_link_joint
- removed joint RFinger12_link_RFinger13_link_joint
- removed joint RFinger21_link_RFinger22_link_joint
- removed joint RFinger22_link_RFinger23_link_joint
- removed joint RFinger31_link_RFinger32_link_joint
- removed joint RFinger32_link_RFinger33_link_joint
- removed joint RFinger41_link_RFinger42_link_joint
- removed joint RFinger42_link_RFinger43_link_joint
- removed joint RForeArm_RElbowRoll_milky_joint
- removed joint RForeArm_r_wrist_joint
- removed joint RShoulder_RBicep_joint
- removed joint RThumb1_link_RThumb2_link_joint
- removed joint Tibia_Pelvis_joint
- removed joint Tibia_WheelB_link_joint
- removed joint Tibia_WheelFL_link_joint
- removed joint Tibia_WheelFR_link_joint
- removed joint Tibia_sick_laser_front_joint
- removed joint Tibia_sick_laser_rear_joint
- removed joint base_footprint_Tibia_joint
- removed joint base_link_base_footprint_joint
- removed joint l_wrist_LFinger11_link_joint
- removed joint l_wrist_LFinger21_link_joint
- removed joint l_wrist_LFinger31_link_joint
- removed joint l_wrist_LFinger41_link_joint
- removed joint l_wrist_LThumb1_link_joint
- removed joint l_wrist_l_gripper_joint
- removed joint r_wrist_RFinger11_link_joint
- removed joint r_wrist_RFinger21_link_joint
- removed joint r_wrist_RFinger31_link_joint
- removed joint r_wrist_RFinger41_link_joint
- removed joint r_wrist_RHandTouchBack_frame_joint
- removed joint r_wrist_RThumb1_link_joint
- removed joint r_wrist_r_gripper_joint
- removed joint torso_LShoulder_joint
- removed joint torso_Neck_joint
- removed joint torso_RShoulder_joint
- added joint AccelerometerBase_sensor_fixedjoint: type fixed, parent Tibia, child ImuBaseAccelerometer_frame, origin xyz=0.0147 -0.0017 -0.26319
- added joint Accelerometer_sensor_fixedjoint: type fixed, parent torso, child ImuTorsoAccelerometer_frame, origin xyz=0.00239 -0.03575 0.14526
- added joint Bumper/Back_sensor_fixedjoint: type fixed, parent Tibia, child BumperB_frame, origin xyz=-0.251 0 -0.264 rpy=0 0 -3.14159
- added joint Bumper/FrontLeft_sensor_fixedjoint: type fixed, parent Tibia, child BumperFL_frame, origin xyz=0.129 0.227 -0.264 rpy=0 0 -5.794325
- added joint Bumper/FrontRight_sensor_fixedjoint: type fixed, parent Tibia, child BumperFR_frame, origin xyz=0.129 -0.227 -0.264 rpy=0 0 -0.48886
- added joint CameraBottom_optical_frame_fixedjoint: type fixed, parent CameraBottom_frame, child CameraBottom_optical_frame, origin rpy=-1.570796 0 -1.570796
- added joint CameraBottom_sensor_fixedjoint: type fixed, parent Head, child CameraBottom_frame, origin xyz=0.09262 0 0.06177 rpy=0 0.698132 0
- added joint CameraDepth_optical_frame_fixedjoint: type fixed, parent CameraDepth_frame, child CameraDepth_optical_frame, origin rpy=-1.570796 0 -1.570796
- added joint CameraDepth_sensor_fixedjoint: type fixed, parent Head, child CameraDepth_frame, origin xyz=0.05138 0.039 0.1194
- added joint CameraTop_optical_frame_fixedjoint: type fixed, parent CameraTop_frame, child CameraTop_optical_frame, origin rpy=-1.570796 0 -1.570796
- added joint CameraTop_sensor_fixedjoint: type fixed, parent Head, child CameraTop_frame, origin xyz=0.08601 0 0.16284
- added joint ChestBoard/Button_sensor_fixedjoint: type fixed, parent torso, child ChestButton_frame, origin xyz=0.049871 0.001588 0.194163
- added joint Gyrometer_sensor_fixedjoint: type fixed, parent torso, child ImuTorsoGyrometer_frame, origin xyz=0.00204 -0.03491 0.12941
- added joint Head/Touch/Front_sensor_fixedjoint: type fixed, parent Head, child HeadTouchFront_frame, origin xyz=0.028175 0 0.21267 rpy=0 0.20944 0
- added joint Head/Touch/Middle_sensor_fixedjoint: type fixed, parent Head, child HeadTouchMiddle_frame, origin xyz=0.0041 0 0.2159 rpy=0 6.248279 0
- added joint Head/Touch/Rear_sensor_fixedjoint: type fixed, parent Head, child HeadTouchRear_frame, origin xyz=-0.03376 0 0.21052 rpy=0 5.969026 0
- added joint HeadPitch: type revolute, parent Neck, child Head, axis 0 1 0, limit lower=-0.706858 upper=0.637045 effort=1000 velocity=1000
- added joint HeadPitch_ears_joint: type fixed, parent Head, child HeadPitch_ears
- added joint HeadPitch_milky_joint: type fixed, parent Head, child HeadPitch_milky
- added joint HeadPitch_shiny_joint: type fixed, parent Head, child HeadPitch_shiny
- added joint HeadYaw: type revolute, parent torso, child Neck, origin xyz=-0.038 0 0.3089, axis 0 0 1, limit lower=-2.08567 upper=2.08567 effort=1000 velocity=1000
- added joint HipPitch: type revolute, parent Pelvis, child Hip, origin xyz=0 0 0.268, axis 0 -1 0, limit lower=-1.03847 upper=1.03847 effort=1000 velocity=1000
- added joint HipPitch_shiny_joint: type fixed, parent Pelvis, child HipPitch_shiny
- added joint HipRoll: type revolute, parent Hip, child torso, origin xyz=-2E-05 0 0.079, axis -1 0 0, limit lower=-0.514872 upper=0.514872 effort=1000 velocity=1000
- added joint KneePitch: type revolute, parent Tibia, child Pelvis, axis 0 -1 0, limit lower=-0.514872 upper=0.514872 effort=1000 velocity=1000
- added joint KneePitch_milky_joint: type fixed, parent Tibia, child KneePitch_milky
- added joint LElbowRoll: type revolute, parent LElbow, child LForeArm, axis 0 0 1, limit lower=-1.56207 upper=-0.008727 effort=1000 velocity=1000
- added joint LElbowRoll_milky_joint: type fixed, parent LForeArm, child LElbowRoll_milky
- added joint LElbowYaw: type revolute, parent LBicep, child LElbow, origin xyz=0.1812 0.015 0.00013 rpy=0 6.126106 0, axis 1 0 0, limit lower=-2.08567 upper=2.08567 effort=1000 velocity=1000
- added joint LFinger11: type revolute, parent l_wrist, child LFinger11_link, origin xyz=0.0821 -0.0268 0.004 rpy=-4.539165 1.04064 -0.033433, axis 0 0 1, limit lower=0 upper=0.872665 effort=1000 velocity=1000
- added joint LFinger12: type revolute, parent LFinger11_link, child LFinger12_link, origin xyz=0.018 0 0 rpy=0 0 -1.0472, axis 0 0 1, limit lower=0 upper=0.872665 effort=1000 velocity=1000
- added joint LFinger13: type revolute, parent LFinger12_link, child LFinger13_link, origin xyz=0.018 0 0 rpy=0 0 -1.0472, axis 0 0 1, limit lower=0 upper=0.872665 effort=1000 velocity=1000
- added joint LFinger21: type revolute, parent l_wrist, child LFinger21_link, origin xyz=0.0873 -0.0073 0.006 rpy=-4.712385 1.0472 -0.061086, axis 0 0 1, limit lower=0 upper=0.872665 effort=1000 velocity=1000
- added joint LFinger22: type revolute, parent LFinger21_link, child LFinger22_link, origin xyz=0.018 0 0 rpy=0 0 -1.0472, axis 0 0 1, limit lower=0 upper=0.872665 effort=1000 velocity=1000
- added joint LFinger23: type revolute, parent LFinger22_link, child LFinger23_link, origin xyz=0.018 0 0 rpy=0 0 -1.0472, axis 0 0 1, limit lower=0 upper=0.872665 effort=1000 velocity=1000
- added joint LFinger31: type revolute, parent l_wrist, child LFinger31_link, origin xyz=0.0833 0.0123 0.004 rpy=-4.816825 1.04483 -0.029314, axis 0 0 1, limit lower=0 upper=0.872665 effort=1000 velocity=1000
- added joint LFinger32: type revolute, parent LFinger31_link, child LFinger32_link, origin xyz=0.018 0 0 rpy=0 0 -1.0472, axis 0 0 1, limit lower=0 upper=0.872665 effort=1000 velocity=1000
- added joint LFinger33: type revolute, parent LFinger32_link, child LFinger33_link, origin xyz=0.018 0 0 rpy=0 0 -1.0472, axis 0 0 1, limit lower=0 upper=0.872665 effort=1000 velocity=1000
- added joint LFinger41: type revolute, parent l_wrist, child LFinger41_link, origin xyz=0.074 0.0309 0 rpy=-4.885615 1.04064 -6.214846, axis 0 0 1, limit lower=0 upper=0.872665 effort=1000 velocity=1000
- added joint LFinger42: type revolute, parent LFinger41_link, child LFinger42_link, origin xyz=0.018 0 0 rpy=0 0 -1.0472, axis 0 0 1, limit lower=0 upper=0.872665 effort=1000 velocity=1000
- added joint LFinger43: type revolute, parent LFinger42_link, child LFinger43_link, origin xyz=0.018 0 0 rpy=0 0 -1.0472, axis 0 0 1, limit lower=0 upper=0.872665 effort=1000 velocity=1000
- added joint LHand: type revolute, parent l_wrist, child l_gripper, origin xyz=0.025 0 0, axis 1 0 0, limit lower=0.02 upper=0.98 effort=1000 velocity=1000
- added joint LHand/Touch/Back_sensor_fixedjoint: type fixed, parent l_wrist, child LHandTouchBack_frame, origin xyz=0.0523 0 0.0304 rpy=0 4.712389 -1.570786
- added joint LShoulderPitch: type revolute, parent torso, child LShoulder, origin xyz=-0.057 0.14974 0.22582, axis 0 1 0, limit lower=-2.08567 upper=2.08567 effort=1000 velocity=1000
- added joint LShoulderRoll: type revolute, parent LShoulder, child LBicep, axis 0 0 1, limit lower=0.008727 upper=1.56207 effort=1000 velocity=1000
- added joint LShoulderRoll_shiny_joint: type fixed, parent LBicep, child LShoulderRoll_shiny
- added joint LThumb1: type revolute, parent l_wrist, child LThumb1_link, origin xyz=0.0482 -0.0357 -0.0199 rpy=-2.55836 0.80626 -5.749207, axis 0 0 1, limit lower=0 upper=0.872665 effort=1000 velocity=1000
- added joint LThumb2: type revolute, parent LThumb1_link, child LThumb2_link, origin xyz=0.022 0 0 rpy=0 0 -1.0472, axis 0 0 1, limit lower=0 upper=0.872665 effort=1000 velocity=1000
- added joint LWristYaw: type revolute, parent LForeArm, child l_wrist, origin xyz=0.15 0 0, axis 1 0 0, limit lower=-1.82387 upper=1.82387 effort=1000 velocity=1000
- added joint LaserSensor/Front_projected_sensor_fixedjoint: type fixed, parent Tibia, child SurroundingFrontLaser_frame, origin xyz=0.0562 0 -0.334
- added joint LaserSensor/Front_sensor_fixedjoint: type fixed, parent Tibia, child SurroundingFrontLaser_device_frame, origin xyz=0.0562 0 -0.0692 rpy=0 0.349066 0
- added joint LaserSensor/Left_projected_sensor_fixedjoint: type fixed, parent Tibia, child SurroundingLeftLaser_frame, origin xyz=-0.018 0.0899 -0.334 rpy=0 0 -4.525905
- added joint LaserSensor/Left_sensor_fixedjoint: type fixed, parent Tibia, child SurroundingLeftLaser_device_frame, origin xyz=-0.018 0.0899 -0.0759 rpy=0 0.349066 -4.712386
- added joint LaserSensor/Right_projected_sensor_fixedjoint: type fixed, parent Tibia, child SurroundingRightLaser_frame, origin xyz=-0.018 -0.0899 -0.334 rpy=0 0 -1.75728
- added joint LaserSensor/Right_sensor_fixedjoint: type fixed, parent Tibia, child SurroundingRightLaser_device_frame, origin xyz=-0.018 -0.0899 -0.0759 rpy=0 0.349066 -1.5708
- added joint LaserSensor/Shovel_sensor_fixedjoint: type fixed, parent Tibia, child ShovelLaser_frame, origin xyz=0.0562 0 -0.0692 rpy=0 0.349066 0
- added joint LaserSensor/VerticalLeft_sensor_fixedjoint: type fixed, parent Tibia, child VerticalLeftLaser_frame, origin xyz=0.0562 0 -0.0692 rpy=0 0.349066 0
- added joint LaserSensor/VerticalRight_sensor_fixedjoint: type fixed, parent Tibia, child VerticalRightLaser_frame, origin xyz=0.0562 0 -0.0692 rpy=0 0.349066 0
- added joint RElbowRoll: type revolute, parent RElbow, child RForeArm, axis 0 0 1, limit lower=0.008727 upper=1.56207 effort=1000 velocity=1000
- added joint RElbowRoll_milky_joint: type fixed, parent RForeArm, child RElbowRoll_milky
- added joint RElbowYaw: type revolute, parent RBicep, child RElbow, origin xyz=0.1812 -0.015 0.00013 rpy=0 6.126106 0, axis 1 0 0, limit lower=-2.08567 upper=2.08567 effort=1000 velocity=1000
- added joint RFinger11: type revolute, parent r_wrist, child RFinger11_link, origin xyz=0.0821 0.0268 0.004 rpy=-4.885615 1.04064 -6.249752, axis 0 0 1, limit lower=0 upper=0.872665 effort=1000 velocity=1000
- added joint RFinger12: type revolute, parent RFinger11_link, child RFinger12_link, origin xyz=0.018 0 0 rpy=0 0 -1.0472, axis 0 0 1, limit lower=0 upper=0.872665 effort=1000 velocity=1000
- added joint RFinger13: type revolute, parent RFinger12_link, child RFinger13_link, origin xyz=0.018 0 0 rpy=0 0 -1.0472, axis 0 0 1, limit lower=0 upper=0.872665 effort=1000 velocity=1000
- added joint RFinger21: type revolute, parent r_wrist, child RFinger21_link, origin xyz=0.0873 0.0073 0.006 rpy=-4.712386 1.0472 -6.222099, axis 0 0 1, limit lower=0 upper=0.872665 effort=1000 velocity=1000
- added joint RFinger22: type revolute, parent RFinger21_link, child RFinger22_link, origin xyz=0.018 0 0 rpy=0 0 -1.0472, axis 0 0 1, limit lower=0 upper=0.872665 effort=1000 velocity=1000
- added joint RFinger23: type revolute, parent RFinger22_link, child RFinger23_link, origin xyz=0.018 0 0 rpy=0 0 -1.0472, axis 0 0 1, limit lower=0 upper=0.872665 effort=1000 velocity=1000
- added joint RFinger31: type revolute, parent r_wrist, child RFinger31_link, origin xyz=0.0833 -0.0123 0.004 rpy=-4.607955 1.04483 -6.253869, axis 0 0 1, limit lower=0 upper=0.872665 effort=1000 velocity=1000
- added joint RFinger32: type revolute, parent RFinger31_link, child RFinger32_link, origin xyz=0.018 0 0 rpy=0 0 -1.0472, axis 0 0 1, limit lower=0 upper=0.872665 effort=1000 velocity=1000
- added joint RFinger33: type revolute, parent RFinger32_link, child RFinger33_link, origin xyz=0.018 0 0 rpy=0 0 -1.0472, axis 0 0 1, limit lower=0 upper=0.872665 effort=1000 velocity=1000
- added joint RFinger41: type revolute, parent r_wrist, child RFinger41_link, origin xyz=0.074 -0.0309 0 rpy=-4.539165 1.04064 -0.06834, axis 0 0 1, limit lower=0 upper=0.872665 effort=1000 velocity=1000
- added joint RFinger42: type revolute, parent RFinger41_link, child RFinger42_link, origin xyz=0.018 0 0 rpy=0 0 -1.0472, axis 0 0 1, limit lower=0 upper=0.872665 effort=1000 velocity=1000
- added joint RFinger43: type revolute, parent RFinger42_link, child RFinger43_link, origin xyz=0.018 0 0 rpy=0 0 -1.0472, axis 0 0 1, limit lower=0 upper=0.872665 effort=1000 velocity=1000
- added joint RHand: type revolute, parent r_wrist, child r_gripper, origin xyz=0.025 0 0, axis 1 0 0, limit lower=0.02 upper=0.98 effort=1000 velocity=1000
- added joint RHand/Touch/Back_sensor_fixedjoint: type fixed, parent r_wrist, child RHandTouchBack_frame, origin xyz=0.0523 0 0.0304 rpy=0 4.712389 -1.570786
- added joint RShoulderPitch: type revolute, parent torso, child RShoulder, origin xyz=-0.057 -0.14974 0.22582, axis 0 1 0, limit lower=-2.08567 upper=2.08567 effort=1000 velocity=1000
- added joint RShoulderRoll: type revolute, parent RShoulder, child RBicep, axis 0 0 1, limit lower=-1.56207 upper=-0.008727 effort=1000 velocity=1000
- added joint RShoulderRoll_shiny_joint: type fixed, parent RBicep, child RShoulderRoll_shiny
- added joint RThumb1: type revolute, parent r_wrist, child RThumb1_link, origin xyz=0.0482 0.0357 -0.0199 rpy=-0.58323 0.80626 -0.533978, axis 0 0 1, limit lower=0 upper=0.872665 effort=1000 velocity=1000
- added joint RThumb2: type revolute, parent RThumb1_link, child RThumb2_link, origin xyz=0.022 0 0 rpy=0 0 -1.0472, axis 0 0 1, limit lower=0 upper=0.872665 effort=1000 velocity=1000
- added joint RWristYaw: type revolute, parent RForeArm, child r_wrist, origin xyz=0.15 0 0, axis 1 0 0, limit lower=-1.82387 upper=1.82387 effort=1000 velocity=1000
- added joint Sonar/Back_sensor_fixedjoint: type fixed, parent Tibia, child SonarBack_frame, origin xyz=-0.0718 0 -0.0534 rpy=0 6.073747 -3.14159
- added joint Sonar/Front_sensor_fixedjoint: type fixed, parent Tibia, child SonarFront_frame, origin xyz=0.0699 0 -0.1023 rpy=0 5.960327 0
- added joint SpeakerLeft_sensor_fixedjoint: type fixed, parent Head, child LSpeaker_frame
- added joint SpeakerRight_sensor_fixedjoint: type fixed, parent Head, child RSpeaker_frame
- added joint Tablet_sensor_fixedjoint: type fixed, parent torso, child Tablet_frame, origin xyz=0.083925 0 0.20151 rpy=0 5.759586 0
- added joint Torso_shiny_joint: type fixed, parent torso, child Torso_shiny, origin xyz=0 0 0.0695
- added joint Torso_transparent_joint: type fixed, parent torso, child Torso_transparent, origin xyz=0 0 0.0695
- added joint WheelB: type continuous, parent Tibia, child WheelB_link, origin xyz=-0.17 0 -0.264 rpy=0 0 -3.14159, axis 1 0 0
- added joint WheelFL: type continuous, parent Tibia, child WheelFL_link, origin xyz=0.09 0.155 -0.264 rpy=0 0 -5.208015, axis 1 0 0
- added joint WheelFR: type continuous, parent Tibia, child WheelFR_link, origin xyz=0.09 -0.155 -0.264 rpy=0 0 -1.07517, axis 1 0 0
- added joint base_footprint_joint: type fixed, parent base_footprint, child Tibia, origin xyz=0 0 0.334
- added joint base_link_joint: type fixed, parent base_link, child base_footprint
- added joint sick_laser_front: type fixed, parent Tibia, child sick_laser_front, origin xyz=0.245 0 -0.1
- added joint sick_laser_rear: type fixed, parent Tibia, child sick_laser_rear, origin xyz=-0.245 0 -0.1 rpy=0 0 -3.141593
